File: PCB/KiCAD_RaumluftWaechter_V1.00_CC_BY-NC-SA_4.0/RaumluftWaechter.kicad_pcb (KiCad board)
At the start: 2 copper layers, 90 x 140 mm, 66 parts, among them J1 Barrel_Jack_Switch, J2 SD_Card_mod, J3 Conn_01x04_Female, Q1 BSS138BKS, SW1 SW_Push, U2 LM1117-3.3, U4 SCD30, U5 DS3231M, U6 74LVC125

Commit message: minor update of schematic, PCB and ibom
Parts:
- R6: value 10K -> 6.8k - 10k
- RN1: value R_Pack04 -> 3.3k
Connections:
- U2 pad 4: /VCC33 -> (no net)
